File: KiCAD/X68k-3mode-fdd-adapter/X68k-3mode-fdd-adapter.kicad_pcb (KiCad board)
At the start: 4 copper layers, 129 x 100 mm, 134 parts, among them J1001 Barrel_Jack_Switch, J1002 USB_C_Receptacle_USB2.0_16P, J101 4pin, J102 Conn_02x06_Odd_Even, J103 Conn_01x02, J104 Conn_01x04, J105 Conn_01x02, J106 Conn_02x17_Odd_Even, J107 Conn_02x17_Odd_Even, J108 Conn_02x17_Odd_Even, Q1001 FDS4935A, Q1002 FDS4935A, Q1003 FDS4935A, Q101 DTC143Z, Q102 2SC2712, Q201 BSS138, Q301 BSS138, Q401 BSS138, Q501 BSS138, Q601 BSS138, Q701 BSS138, Q801 BSS138, Q901 BSS138, SW101 SW_DIP_x04, SW102 RESET, U1001 K7805M-1000R3, U1002 MCP1792x-5002xCB, U101 INA3221AIRGVR, U102 SLG46826G(V2), U103 SLG46826G(V2), U104 CH32X035C8T6, U105 SLG46826G(V2)

Commit message: 試作基板の発注
Parts:
- moved D101 4.60 mm to (167.5, 136.5)
- moved Q102 4.60 mm to (168.0, 140.5)
- moved R107 4.60 mm to (165.0, 140.5)
- moved BZ101 4.60 mm to (175.3, 138.7)
Routing:
- net VDD_MCU: track 142.1 -> 148.9 mm
- net /BUZZER: track 64.5 -> 65.5 mm
- net /DIPSW_MODESEL_POL: track 35.0 -> 34.2 mm
- added copper zone on In1.Cu, net GND
Other:
- board text added: "+12V GND GND +5V"
- board text added: "DSEL 0 DSEL 1 MSEL POL PD +12V"
- board text added: "Developed by @kunichiko and @kani7. September 2025 (${REVISION})"
- board text added: "I2C SDA I2C SCL LED DATA OPTION VDD FDD IF VDD MCU"
- board text added: "I2C SDA I2C SCL VDD MCU GND"
- board text removed: "Developed by @kunichiko and @kani7. September 2025 (V2.0.0)"
