File: KiCAD/X68k-3mode-fdd-adapter/serial_leds.kicad_sch (KiCad schematic)
At the start: 5 parts, among them J101 Conn_01x03_Pin

Commit message: DRCエラー修正
Parts:
- D1101: renamed from D101; symbol X68k-lib:SK6812MINI-HS -> x68000-ext:SK6812MINI-HS
- D1102: renamed from D102; symbol X68k-lib:SK6812MINI-HS -> x68000-ext:SK6812MINI-HS
- D1103: renamed from D1101; symbol X68k-lib:SK6812MINI-HS -> x68000-ext:SK6812MINI-HS
- D1104: renamed from D1102; symbol X68k-lib:SK6812MINI-HS -> x68000-ext:SK6812MINI-HS
- renumbered J101 to J1101
Connections:
- net +5V renamed VDD_MCU
Changed lines of the file:
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@@
 	)
 	(symbol
-		(lib_id "X68k-lib:SK6812MINI-HS")
+		(lib_id "x68000-ext:SK6812MINI-HS")
 		(at 144.78 102.87 0)
 		(unit 1)
@@
 		(on_board yes)
 		(dnp no)
-		(property "Reference" "D1101"
+		(property "Reference" "D1103"
 			(at 149.86 91.948 0)
 			(effects
@@
 			(project "X68k-3mode-fdd-adapter"
 				(path "/13b3a4ee-84d6-44b3-962d-9cf7c36d7564/31293df3-a871-47ca-8f5f-1d9e3b862849"
-					(reference "D1101")
-					(unit 1)
-				)
-			)
-		)
-	)
-	(symbol
-		(lib_id "X68k-lib:SK6812MINI-HS")
+					(reference "D1103")
+					(unit 1)
+				)
+			)
+		)
+	)
+	(symbol
+		(lib_id "x68000-ext:SK6812MINI-HS")
 		(at 83.82 102.87 0)
 		(unit 1)
@@
 		(on_board yes)
 		(dnp no)
-		(property "Reference" "D101"
+		(property "Reference" "D1101"
 			(at 88.9 91.948 0)
 			(effects
@@
 			(project "X68k-3mode-fdd-adapter"
 				(path "/13b3a4ee-84d6-44b3-962d-9cf7c36d7564/31293df3-a871-47ca-8f5f-1d9e3b862849"
-					(reference "D101")
+					(reference "D1101")
 					(unit 1)
 				)
@@
 		(dnp no)
 		(fields_autoplaced yes)
-		(property "Reference" "#PWR01103"
+		(property "Reference" "#PWR01109"
 			(at 144.78 119.38 0)
 			(effects
@@
 			(project "X68k-3mode-fdd-adapter"
 				(path "/13b3a4ee-84d6-44b3-962d-9cf7c36d7564/31293df3-a871-47ca-8f5f-1d9e3b862849"
-					(reference "#PWR01103")
+					(reference "#PWR01109")
 					(unit 1)
 				)
@@
 		(dnp no)
 		(fields_autoplaced yes)
-		(property "Reference" "#PWR0111"
+		(property "Reference" "#PWR01102"
 			(at 71.12 93.98 0)
 			(effects
@@
 			(project "X68k-3mode-fdd-adapter"
 				(path "/13b3a4ee-84d6-44b3-962d-9cf7c36d7564/31293df3-a871-47ca-8f5f-1d9e3b862849"
-					(reference "#PWR0111")
+					(reference "#PWR01102")
 					(unit 1)
 				)
@@
 		(dnp no)
 		(fields_autoplaced yes)
-		(property "Reference" "#PWR0107"
+		(property "Reference" "#PWR01101"
 			(at 71.12 77.47 0)
 			(effects
@@
 			)
 		)
-		(property "Value" "+5V"
+		(property "Value" "VDD_MCU"
 			(at 71.12 68.58 0)
 			(effects
@@
 			(project "X68k-3mode-fdd-adapter"
 				(path "/13b3a4ee-84d6-44b3-962d-9cf7c36d7564/31293df3-a871-47ca-8f5f-1d9e3b862849"
-					(reference "#PWR0107")
-					(unit 1)
-				)
-			)
-		)
-	)
-	(symbol
-		(lib_id "X68k-lib:SK6812MINI-HS")
+					(reference "#PWR01101")
+					(unit 1)
+				)
+			)
+		)
+	)
+	(symbol
+		(lib_id "x68000-ext:SK6812MINI-HS")
 		(at 171.45 102.87 0)
 		(unit 1)
@@
 		(on_board yes)
 		(dnp no)
-		(property "Reference" "D1102"
+		(property "Reference" "D1104"
 			(at 175.768 92.71 0)
 			(effects
@@
 			(project "X68k-3mode-fdd-adapter"
 				(path "/13b3a4ee-84d6-44b3-962d-9cf7c36d7564/31293df3-a871-47ca-8f5f-1d9e3b862849"
-					(reference "D1102")
+					(reference "D1104")
 					(unit 1)
 				)
@@
 		(dnp no)
 		(fields_autoplaced yes)
-		(property "Reference" "#PWR01104"
+		(property "Reference" "#PWR01110"
 			(at 171.45 119.38 0)
 			(effects
@@
 			(project "X68k-3mode-fdd-adapter"
 				(path "/13b3a4ee-84d6-44b3-962d-9cf7c36d7564/31293df3-a871-47ca-8f5f-1d9e3b862849"
-					(reference "#PWR01104")
+					(reference "#PWR01110")
 					(unit 1)
 				)
@@
 		(dnp no)
 		(fields_autoplaced yes)
-		(property "Reference" "#PWR0117"
+		(property "Reference" "#PWR01107"
 			(at 83.82 119.38 0)
 			(effects
@@
 			(project "X68k-3mode-fdd-adapter"
 				(path "/13b3a4ee-84d6-44b3-962d-9cf7c36d7564/31293df3-a871-47ca-8f5f-1d9e3b862849"
-					(reference "#PWR0117")
+					(reference "#PWR01107")
 					(unit 1)
 				)
@@
 		(dnp no)
 		(fields_autoplaced yes)
-		(property "Reference" "#PWR0112"
+		(property "Reference" "#PWR01103"
 			(at 83.82 97.79 0)
 			(effects
@@
 			)
 		)
-		(property "Value" "+5V"
+		(property "Value" "VDD_MCU"
 			(at 83.82 88.9 0)
 			(effects
@@
 			(project "X68k-3mode-fdd-adapter"
 				(path "/13b3a4ee-84d6-44b3-962d-9cf7c36d7564/31293df3-a871-47ca-8f5f-1d9e3b862849"
-					(reference "#PWR0112")
+					(reference "#PWR01103")
 					(unit 1)
 				)
@@
 		(dnp no)
 		(fields_autoplaced yes)
-		(property "Reference" "#PWR01102"
+		(property "Reference" "#PWR01106"
 			(at 171.45 97.79 0)
 			(effects
@@
 			)
 		)
-		(property "Value" "+5V"
+		(property "Value" "VDD_MCU"
 			(at 171.45 88.9 0)
 			(effects
@@
 			(project "X68k-3mode-fdd-adapter"
 				(path "/13b3a4ee-84d6-44b3-962d-9cf7c36d7564/31293df3-a871-47ca-8f5f-1d9e3b862849"
-					(reference "#PWR01102")
+					(reference "#PWR01106")
 					(unit 1)
 				)
@@
 		(dnp no)
 		(fields_autoplaced yes)
-		(property "Reference" "#PWR0118"
+		(property "Reference" "#PWR01108"
 			(at 110.49 119.38 0)
 			(effects
@@
 			(project "X68k-3mode-fdd-adapter"
 				(path "/13b3a4ee-84d6-44b3-962d-9cf7c36d7564/31293df3-a871-47ca-8f5f-1d9e3b862849"
-					(reference "#PWR0118")
+					(reference "#PWR01108")
 					(unit 1)
 				)
@@
 		(dnp no)
 		(fields_autoplaced yes)
-		(property "Reference" "#PWR01101"
+		(property "Reference" "#PWR01105"
 			(at 144.78 97.79 0)
 			(effects
@@
 			)
 		)
-		(property "Value" "+5V"
+		(property "Value" "VDD_MCU"
 			(at 144.78 88.9 0)
 			(effects
@@
 			(project "X68k-3mode-fdd-adapter"
 				(path "/13b3a4ee-84d6-44b3-962d-9cf7c36d7564/31293df3-a871-47ca-8f5f-1d9e3b862849"
-					(reference "#PWR01101")
+					(reference "#PWR01105")
 					(unit 1)
 				)
@@
 		(dnp no)
 		(fields_autoplaced yes)
-		(property "Reference" "J101"
+		(property "Reference" "J1101"
 			(at 80.01 78.7399 0)
 			(effects
@@
 			(project "X68k-3mode-fdd-adapter"
 				(path "/13b3a4ee-84d6-44b3-962d-9cf7c36d7564/31293df3-a871-47ca-8f5f-1d9e3b862849"
-					(reference "J101")
+					(reference "J1101")
 					(unit 1)
 				)
@@
 		(dnp no)
 		(fields_autoplaced yes)
-		(property "Reference" "#PWR0113"
+		(property "Reference" "#PWR01104"
 			(at 110.49 97.79 0)
 			(effects
@@
 			)
 		)
-		(property "Value" "+5V"
+		(property "Value" "VDD_MCU"
 			(at 110.49 88.9 0)
 			(effects
@@
 			(project "X68k-3mode-fdd-adapter"
 				(path "/13b3a4ee-84d6-44b3-962d-9cf7c36d7564/31293df3-a871-47ca-8f5f-1d9e3b862849"
-					(reference "#PWR0113")
-					(unit 1)
-				)
-			)
-		)
-	)
-	(symbol
-		(lib_id "X68k-lib:SK6812MINI-HS")
+					(reference "#PWR01104")
+					(unit 1)
+				)
+			)
+		)
+	)
+	(symbol
+		(lib_id "x68000-ext:SK6812MINI-HS")
 		(at 110.49 102.87 0)
 		(unit 1)
@@
 		(on_board yes)
 		(dnp no)
-		(property "Reference" "D102"
+		(property "Reference" "D1102"
 			(at 114.808 92.71 0)
 			(effects
@@
 			(project "X68k-3mode-fdd-adapter"
 				(path "/13b3a4ee-84d6-44b3-962d-9cf7c36d7564/31293df3-a871-47ca-8f5f-1d9e3b862849"
-					(reference "D102")
-					(unit 1)
-				)
+					(reference "D1102")
+					(unit 1)
+				)

Commit message: PCBの配線完了
Parts:
- removed J1101: Conn_01x03_Pin, Connector_PinHeader_2.54mm:PinHeader_1x03_P2.54mm_Vertical, symbol Connector:Conn_01x03_Pin

Commit message: フロントパネルを作り始めた
Changed lines of the file:
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@@
 			)
 		)
-		(property "Description" "RGB LED with integrated controller"
-			(at 144.78 102.87 0)
-			(effects
-				(font
-					(size 1.27 1.27)
-				)
-				(hide yes)
+		(property "Description" "ACCESS B"
+			(at 144.78 85.09 0)
+			(effects
+				(font
+					(size 1.27 1.27)
+				)
 			)
 		)
@@
 					(size 1.27 1.27)
 				)
+				(hide yes)
 			)
 		)
@@
 			)
 		)
-		(property "Description" "RGB LED with integrated controller"
-			(at 83.82 102.87 0)
-			(effects
-				(font
-					(size 1.27 1.27)
-				)
-				(hide yes)
+		(property "Description" "ACCESS A"
+			(at 83.82 84.836 0)
+			(effects
+				(font
+					(size 1.27 1.27)
+				)
 			)
 		)
@@
 					(size 1.27 1.27)
 				)
+				(hide yes)
 			)
 		)
@@
 			)
 		)
-		(property "Description" "RGB LED with integrated controller"
-			(at 171.45 102.87 0)
-			(effects
-				(font
-					(size 1.27 1.27)
-				)
-				(hide yes)
+		(property "Description" "EJECT B"
+			(at 171.45 85.344 0)
+			(effects
+				(font
+					(size 1.27 1.27)
+				)
 			)
 		)
@@
 					(size 1.27 1.27)
 				)
+				(hide yes)
 			)
 		)
@@
 			)
 		)
-		(property "Description" "RGB LED with integrated controller"
-			(at 110.49 102.87 0)
-			(effects
-				(font
-					(size 1.27 1.27)
-				)
-				(hide yes)
+		(property "Description" "EJECT A"
+			(at 110.49 84.836 0)
+			(effects
+				(font
+					(size 1.27 1.27)
+				)
 			)
 		)
 		(property "LCSC" "C2922787"
-			(at 110.49 102.87 0)
-			(effects
-				(font
-					(size 1.27 1.27)
-				)
-			)
-		)
+			(at 105.41 105.41 0)
+			(effects
+				(font
+					(size 1.27 1.27)
+				)
+				(hide yes)
+			)
+		)

Commit message: V2.1.0の基板を引き切った
Parts:
- removed D1101, D1102, D1103, D1104: SK6812MINI, x68k-lib:SK6812MINI-HS, symbol x68000-ext:SK6812MINI-HS
- added D1501, D1502, D1503, D1504: WS2812B-2020, LED_SMD:LED_WS2812B-2020_PLCC4_2.0x2.0mm, symbol LED:WS2812B-2020
Connections:
- net GND: now also D1501.2 (VSS), D1502.2 (VSS), D1503.2 (VSS), D1504.2 (VSS)
- net LED_DATA: now also D1501.3 (DIN)
- net VDD_MCU: now also D1501.4 (VDD), D1502.4 (VDD), D1503.4 (VDD), D1504.4 (VDD)
- new net: D1502.1 (DOUT), D1503.3 (DIN)
- new net: D1501.1 (DOUT), D1502.3 (DIN)
- new net: D1503.1 (DOUT), D1504.3 (DIN)
