File: KiCAD/X68k-3mode-fdd-adapter/open_drain_buffer.kicad_sch (KiCad schematic)
At the start: 3 parts, among them Q201 BSS138

Commit message: フットプリントを一通り割り当てた
Parts:
- R201, R202: footprint (none) -> Resistor_SMD:R_0603_1608Metric
Changed lines of the file:
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@@
 			)
 		)
-		(property "Footprint" ""
+		(property "Footprint" "Resistor_SMD:R_0603_1608Metric"
 			(at 127 97.79 0)
 			(effects
@@
 			)
 		)
-		(property "Footprint" ""
+		(property "Footprint" "Resistor_SMD:R_0603_1608Metric"
 			(at 132.08 100.33 0)
 			(effects

Commit message: v2.0.1向けの修正を一通り入れたので一旦コミット
Parts:
- R202: value 100 -> 100k
Changed lines of the file:
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@@
 			)
 		)
-		(property "Value" "100"
+		(property "Value" "100k"
 			(at 134.874 98.806 90)
 			(effects
