File: KiCAD/X68k-3mode-fdd-adapter/speaker.kicad_sch (KiCad schematic)
At the start: 6 parts, among them Q1701 2SC2712

Commit message: PCBA発注のために部品番号などを追加した
Parts:
- BZ1701: now not fitted
- Q1701: footprint Package_TO_SOT_SMD:SOT-323_SC-70 -> Package_TO_SOT_SMD:SC-59_Handsoldering
Changed lines of the file:
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@@
-			)
-		)
-		(property "LCIC" ""
-			(at 105.41 96.52 0)
-			(effects
-				(font
-					(size 1.27 1.27)
-				)
-				(hide yes)
 			)
 		)
@@
 		)
 		(property "Description" "Jumper, 2-pole, small symbol, open"
-			(at 109.22 69.85 0)
-			(effects
-				(font
-					(size 1.27 1.27)
-				)
-				(hide yes)
-			)
-		)
-		(property "LCIC" ""
 			(at 109.22 69.85 0)
 			(effects
@@
 			)
 		)
-		(property "LCIC" ""
-			(at 115.57 69.85 0)
-			(effects
-				(font
-					(size 1.27 1.27)
-				)
-				(hide yes)
-			)
-		)
 		(pin "1"
 		)
@@
 			)
 		)
-		(property "LCIC" ""
-			(at 111.76 78.74 90)
-			(effects
-				(font
-					(size 1.27 1.27)
-				)
-				(hide yes)
-			)
-		)
 		(pin "1"
 		)
@@
 			)
 		)
-		(property "Footprint" "Package_TO_SOT_SMD:SOT-323_SC-70"
+		(property "Footprint" "Package_TO_SOT_SMD:SC-59_Handsoldering"
 			(at 118.11 93.345 0)
 			(effects
@@
 		)
 		(property "Description" "0.3A Ic, 20V Vce, NPN Transistor, For Muting and Switching, SOT-323"
-			(at 113.03 91.44 0)
-			(effects
-				(font
-					(size 1.27 1.27)
-				)
-				(hide yes)
-			)
-		)
-		(property "LCIC" ""
 			(at 113.03 91.44 0)
 			(effects
@@
 		(in_bom yes)
 		(on_board yes)
-		(dnp no)
+		(dnp yes)
 		(fields_autoplaced yes)
 		(property "Reference" "BZ1701"
@@
 			(at 124.46 78.74 0)
 			(effects
-				(font
-					(size 1.27 1.27)
-				)
-				(hide yes)
-			)
-		)
-		(property "LCIC" ""
-			(at 124.46 78.74 0)
-			(effects
