File: KiCAD/X68k-3mode-fdd-adapter/usb_pd_pwr.kicad_sch (KiCad schematic)
At the start: 32 parts, among them J1001 Barrel_Jack_Switch, J1002 USB_C_Receptacle_USB2.0_16P, Q1001 FDS4935A, Q1002 FDS4935A, Q1003 FDS4935A, Q1004 DTC143Z, Q1005 DTC143Z, Q1006 DTC143Z, Q1007 FDS4935A, U1001 K7805M-1000R3, U1002 AP2210N-5.0TRG1

Commit message: V2.1.0の基板を引き切った
Parts:
- added C1405, C1406: 1uF, Capacitor_SMD:C_0603_1608Metric_Pad1.08x0.95mm_HandSolder, symbol Device:C_Small
- added U1403: XC6201P332MR-G, Package_TO_SOT_SMD:SOT-23-5_HandSoldering, symbol x68000-ext:XC6201P332MR-G
- renumbered C1003 to C1401, C1004 to C1402, C1001 to C1403, C1002 to C1404, D1001 to D1401, D1005 to D1402, D1004 to D1403, D1003 to D1404, J1002 to J1401, J1001 to J1402, Q1003 to Q1401, Q1001 to Q1402, Q1002 to Q1403, Q1006 to Q1404, Q1004 to Q1405, Q1005 to Q1406, Q1007 to Q1407, R1008 to R1401, R1009 to R1402, R1007 to R1403, R1010 to R1404, R1011 to R1405, R1005 to R1406, R1006 to R1407, R1001 to R1408, R1002 to R1409, R1003 to R1410, R1004 to R1411, R1012 to R1412, R1013 to R1413, U1002 to U1401, U1001 to U1402
Connections:
- net GND: now also C1405.2, C1406.2, U1403.2 (GND)
- net VDD_MCU: now also C1405.1, U1403.1 (VI)
- new net +3.3V: C1406.1, U1403.5 (VO)

Commit message: PCBA発注のために部品番号などを追加した
Parts:
- J1402: LCSC (none) -> C16214
