File: KiCAD/X68k-3mode-fdd-adapter/mounting_hole.kicad_sch (KiCad schematic)
At the start: 12 parts

Commit message: 一部部品が未実装になっていたりしたので修正して出しなおした
Parts:
- H1601, H1602, H1603, H1604, H1605, H1606: now in the parts list
